File: workspace/Battery.kicad_sch (KiCad schematic)
At the start: 11 parts, among them J1 Screw_Terminal_01x02, J2 Conn_01x05

Commit message: Formation 3/4
Parts:
- H1, H2: footprint (none) -> MountingHole:MountingHole_2.7mm
- H3, H4: footprint (none) -> MountingHole:MountingHole_2.7mm_Pad
- J1: footprint (none) -> TerminalBlock_Phoenix:TerminalBlock_Phoenix_MKDS-1,5-2_1x02_P5.00mm_Horizontal
- J2: footprint (none) -> Connector_JST:JST_PH_S5B-PH-K_1x05_P2.00mm_Horizontal
- R1, R2, R3: footprint (none) -> Resistor_SMD:R_0603_1608Metric
- R_SHUNT1: footprint (none) -> Resistor_Shunt:Milliohm_Shunt_2512
- U1: footprint (none) -> Package_DFN_QFN:DFN-8-1EP_3x3mm_P0.5mm_EP1.65x2.38mm_ThermalVias
Connections:
- net at R_SHUNT1.1, U1.1 (SENSE+): now also J1.2 (Pin_2); no longer J1.1 (Pin_1)
- net at R_SHUNT1.2, U1.8 (SENSE-): now also J1.1 (Pin_1); no longer J1.2 (Pin_2)
